Commit message: Add Cheetah CAN protocol

File: test/test_state_publisher.urdf.xacro (robot description, xacro)
@@ -1,45 +1,83 @@
 <?xml version="1.0"?>
 <robot xmlns:xacro="http://www.ros.org/wiki/xacro" name="test_state_publisher_robot">
-    <link name="base_link">
-      <inertial>
-        <origin xyz="0 0 0" rpy="0 0 0"/>
-        <mass value="3.0"/>
-        <inertia ixx="0.001" ixy="0" ixz="0" iyy="0.001" iyz="0" izz="0.001"/>
-      </inertial>
-      <visual name="Cube">
-        <origin xyz="0 0 0" rpy="0 0 0"/>
-        <geometry>
-          <box size="0.24 0.14 0.22"/>
-        </geometry>
-      </visual>
-    </link>
-    <link name="imu">
-      <inertial>
-        <origin xyz="0 0 0" rpy="0 0 0"/>
-        <mass value="0.001"/>
-        <inertia ixx="0.001" ixy="0" ixz="0" iyy="0.001" iyz="0" izz="0.001"/>
-      </inertial>
-    </link>
-    <joint name="imu" type="fixed">
-      <origin xyz="0 0 0" rpy="1.5708 0 1.5708"/>
-      <parent link="base_link"/>
-      <child link="imu"/>
-    </joint>
-    <ros2_control name="pi3hat_hardware_interface" type="system">
+  <link name="base_link">
+    <inertial>
+      <origin xyz="0 0 0" rpy="0 0 0"/>
+      <mass value="3.0"/>
+      <inertia ixx="0.001" ixy="0" ixz="0" iyy="0.001" iyz="0" izz="0.001"/>
+    </inertial>
+    <visual name="Cube">
+      <origin xyz="0 0 0" rpy="0 0 0"/>
+      <geometry>
+        <box size="0.24 0.14 0.22"/>
+      </geometry>
+    </visual>
+  </link>
+  <link name="imu">
+    <inertial>
+      <origin xyz="0 0 0" rpy="0 0 0"/>
+      <mass value="0.001"/>
+      <inertia ixx="0.001" ixy="0" ixz="0" iyy="0.001" iyz="0" izz="0.001"/>
+    </inertial>
+  </link>
+  <joint name="imu" type="fixed">
+    <origin xyz="0 0 0" rpy="1.5708 0 1.5708"/>
+    <parent link="base_link"/>
+    <child link="imu"/>
+  </joint>
+  <ros2_control name="pi3hat_hardware_interface" type="system">
       <hardware>
-        <plugin>pi3hat_hardware_interface/Pi3HatHardwareInterface</plugin>
+          <plugin>pi3hat_hardware_interface/Pi3HatHardwareInterface</plugin>
+          <param name="imu_mounting_deg.yaw">0</param>
+          <param name="imu_mounting_deg.pitch">0</param>
+          <param name="imu_mounting_deg.roll">0</param>
       </hardware>
+      <joint name="joint1">
+          <param name="can_channel">1</param>
+          <param name="can_id">1</param>
+          <param name="can_protocol">"cheetah"</param>
+          <param name="position_scale">95.5</param>
+          <param name="velocity_scale">30.0</param>
+          <param name="effort_scale">18.0</param>
+          <param name="kp_scale">500.0</param>
+          <param name="kd_scale">5.0</param>
+          <param name="axis_direction">-1</param>
+          <param name="position_offset">0.0</param>
+          <command_interface name="position">
+              <param name="min">-1</param>
+              <param name="max">1</param>
+          </command_interface>
+          <command_interface name="velocity">
+              <param name="min">-1</param>
+              <param name="max">1</param>
+          </command_interface>
+          <command_interface name="effort">
+              <param name="min">-1</param>
+              <param name="max">1</param>
+          </command_interface>
+          <command_interface name="kp">
+              <param name="min">-1</param>
+              <param name="max">1</param>
+          </command_interface>
+          <command_interface name="kd">
+              <param name="min">-1</param>
+              <param name="max">1</param>
+          </command_interface>
+          <state_interface name="position"/>
+          <state_interface name="velocity"/>
+          <state_interface name="effort"/>
+      </joint>
       <sensor name="imu_sensor">
-        <state_interface name="orientation.x"/>
-        <state_interface name="orientation.y"/>
-        <state_interface name="orientation.z"/>
-        <state_interface name="orientation.w"/>
-        <state_interface name="angular_velocity.x"/>
-        <state_interface name="angular_velocity.y"/>
-        <state_interface name="angular_velocity.z"/>
-        <state_interface name="linear_acceleration.x"/>
-        <state_interface name="linear_acceleration.y"/>
-        <state_interface name="linear_acceleration.z"/>
+          <state_interface name="orientation.x"/>
+          <state_interface name="orientation.y"/>
+          <state_interface name="orientation.z"/>
+          <state_interface name="orientation.w"/>
+          <state_interface name="angular_velocity.x"/>
+          <state_interface name="angular_velocity.y"/>
+          <state_interface name="angular_velocity.z"/>
+          <state_interface name="linear_acceleration.x"/>
+          <state_interface name="linear_acceleration.y"/>
+          <state_interface name="linear_acceleration.z"/>
       </sensor>
-    </ros2_control>
+  </ros2_control>
 </robot>

Commit message: Update test files and readme

File: test/test_state_publisher.urdf.xacro (robot description, xacro)
@@ -14,4 +14,24 @@
     </visual>
   </link>
+  <link name="link_1">
+    <inertial>
+      <origin xyz="0 0 0" rpy="0 0 0"/>
+      <mass value="3.0"/>
+      <inertia ixx="0.001" ixy="0" ixz="0" iyy="0.001" iyz="0" izz="0.001"/>
+    </inertial>
+    <visual name="Cube">
+      <origin xyz="0 0 0" rpy="0 0 0"/>
+      <geometry>
+        <box size="0.24 0.14 0.22"/>
+      </geometry>
+    </visual>
+  </link>
+  <joint name="joint_1" type="revolute">
+    <origin xyz="0 -0.1 0" rpy="1.5708 1.5708 0"/>
+    <parent link="base_link"/>
+    <child link="link_1"/>
+    <axis xyz="0 0 1.0"/>
+    <limit lower="-1.39626" upper="-0.5236" effort="35.0" velocity="26.0"/>
+  </joint>
   <link name="imu">
     <inertial>
@@ -33,8 +53,8 @@
           <param name="imu_mounting_deg.roll">0</param>
       </hardware>
-      <joint name="joint1">
+      <joint name="joint_1">
           <param name="can_channel">1</param>
           <param name="can_id">1</param>
-          <param name="can_protocol">"cheetah"</param>
+          <param name="can_protocol">cheetah</param>
           <param name="position_scale">95.5</param>
           <param name="velocity_scale">30.0</param>
